File: currentShuntAmpDiscretesRes01/currentShuntAmpDiscretesRes01.sch (KiCad schematic (older format))
At the start: 10 parts, among them Q1 2N3906, Q2 2N3906

Commit message: evolution of currentShuntAmpDiscretes, not working yet
Parts:
- R2: value 1K -> 500
- R3: value 1K -> 0
- R4: value 52.5K -> 174K
- R5: value 240K -> 200K
- R6: value 37.5K -> 26K
- V1: value +12V -> +30V
Connections:
- net Ve1: now reaches Q1.3 (E), R2.2
- net Ve2: now reaches Q2.3 (E), R3.2
Other:
- note added: "+PSPICE \n*.include ../ComponentModels/1n4148.spi\n.include ../ComponentModels/2n3906.spi\n*.include ../ComponentModels/irf4905.spi\n\n.DC I1 -0.5 8.5 0.1 V1 20 40 10 \n// DC analysis for 20, 30 and 40 Volts\n//.DC I1 -0.5 8.5 0.1\n// DC analysis from -0.5 to 8.5 Amps in steps of 0.1 Amp\n\n*.TRAN 0.05us 10ms\n // transient analysis for 10 ms in steps of 0.1 us (10,000 steps)\n.control\nrun\nplot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"
- note added: "Objectives:\nShunt resistor 10 m Ohms\nCurrent unidirectional 8 A\nVout 0 at 0 A, 5V at 8A"
- note removed: "+PSPICE \n*.include ../ComponentModels/1n4148.spi\n.include ../ComponentModels/2n3906.spi\n*.include ../ComponentModels/irf4905.spi\n\n.DC I1 -12 12 0.1\n// DC analysis from 0 to 1 Amps in steps of 1 Amp\n*.TRAN 0.05us 10ms\n // transient analysis for 10 ms in steps of 0.1 us (10,000 steps)\n.control\nrun\nplot VA VK VC Vbase\nplot (VA-VK)\nplot (VA-VK)*23.5+2.15 Vout\nplot (VA-VK)*23.5+2.15-Vout"
- moved on the sheet: I1, Q1, Q2, R1, R2, R3, R4, R5, R6, V1
