File: currentShunt/currentShuntAmpOpAmpUni/currentShuntAmpOpAmpUni.sch (KiCad schematic (older format))
At the start: 11 parts, among them Q1 2N3906, U1 AD822A

Commit message: updated folder structure
Parts:
- D1: value D1N4733 -> 1N4733
Other:
- note added: "+PSPICE \n*.include ../../ComponentModels/1n4148.spi\n.include ../../ComponentModels/2n3906.spi\n.include ../../ComponentModels/ad822a.cir\n.include ../../ComponentModels/1n4733.spi\n\n.DC I1 0 8 0.1 V1 20 40 10 \n*.DC I1 -0.1 0.8 0.01 \n// DC analysis for 20, 30 and 40 Volts\n//.DC I1 -0.5 8.5 0.1\n// DC analysis from -0.5 to 8.5 Amps in steps of 0.1 Amp\n\n*.TRAN 1us 10ms\n // transient analysi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"
- note removed: "+PSPICE \n*.include ../ComponentModels/1n4148.spi\n.include ../ComponentModels/2n3906.spi\n.include ../ComponentModels/ad822a.cir\n*.include ../ComponentModels/irf4905.spi\n.model D1N4733 D(Is=1.214f Rs=1.078 Ikf=0 N=1 Xti=3 Eg=1.11\n+ Cjo=185p M=.3509 Vj=.75 Fc=.5 Bv=5.1 Ibv=.70507\n+ Nbv=.74348 )\n* Motorola pid=1N4733 case=DO-41\n\n.DC I1 0 8 0.1 V1 20 40 10 \n*.DC I1 -0.1 0.8 0.01 \n// DC ana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"
Changed lines of the file:
@@
 	1    0    0    -1
 $EndComp
-Text Notes 4400 3350 0    60   ~ 0
-+PSPICE \n*.include ../ComponentModels/1n4148.spi\n.include ../ComponentModels/2n3906.spi\n.include ../ComponentModels/ad822a.cir\n*.include ../ComponentModels/irf4905.spi\n.model D1N4733 D(Is=1.214f Rs=1.078 Ikf=0 N=1 Xti=3 Eg=1.11\n+ Cjo=185p M=.3509 Vj=.75 Fc=.5  Bv=5.1 Ibv=.70507\n+ Nbv=.74348 )\n* Motorola pid=1N4733 case=DO-41\n\n.DC I1 0 8 0.1  V1 20 40 10 \n*.DC I1 -0.1 0.8 0.01  \n// DC analysis for 20, 30 and 40 Volts\n//.DC I1 -0.5 8.5 0.1\n// DC analysis from -0.5 to 8.5 Amps in steps of 0.1 Amp\n\n*.TRAN 0.05us 10ms\n // transient analysis for 10 ms in steps of 0.1 us (10,000 steps)\n.control\nrun\n*plot Va Ve1 Vk\n*plot (VA-VK)*25+2.693 Vout\n*plot (VA-VK)*25+2.693-Vout\n*plot VA VK  Vbase\n*plot VK-Vref\n*plot Ve1-Vc1 VA-Ve1 VA-Vc1 VK-Vc1\nplot vout\nplot vout-i(v1)*5/8 // voltage error\nplot vout*8/5-i(v1) // ccurrent error\n*plot i1\n
+Text Notes 4550 3700 0    60   ~ 0
++PSPICE \n*.include ../../ComponentModels/1n4148.spi\n.include ../../ComponentModels/2n3906.spi\n.include ../../ComponentModels/ad822a.cir\n.include ../../ComponentModels/1n4733.spi\n\n.DC I1 0 8 0.1  V1 20 40 10 \n*.DC I1 -0.1 0.8 0.01  \n// DC analysis for 20, 30 and 40 Volts\n//.DC I1 -0.5 8.5 0.1\n// DC analysis from -0.5 to 8.5 Amps in steps of 0.1 Amp\n\n*.TRAN 1us 10ms\n // transient analysis for 10 ms in steps of 1 us (10,000 steps)\n.control\nrun\n*plot Va Ve1 Vk\n*plot (VA-VK)*25+2.693 Vout\n*plot (VA-VK)*25+2.693-Vout\n*plot VA VK  Vbase\n*plot VK-Vref\n*plot Ve1-Vc1 VA-Ve1 VA-Vc1 VK-Vc1\nplot vout\nplot vout-i(v1)*5/8 // voltage error\nplot vout*8/5-i(v1) // current error\n*plot i1\n
 Connection ~ 2300 700
 $Comp
@@
 P 3150 1250
 F 0 "D1" H 3150 1350 50  0000 C CNN
-F 1 "D1N4733" H 3150 1150 50  0000 C CNN
+F 1 "1N4733" H 3150 1150 50  0000 C CNN
 F 2 "" H 3150 1250 50  0001 C CNN
 F 3 "" H 3150 1250 50  0001 C CNN
