File: MOSFETdiode/MOSFETdiodeDiscretes/MOSFETdiodeDiscretes.sch (KiCad schematic (older format))
At the start: 13 parts, among them Q1 IRF4905, Q2 2N3906, Q3 2N3906

Commit message: updated for folder restructure
Parts:
- XQ1: renamed from Q1; Spice_Node_Sequence (none) -> 2,1,3
Other:
- note added: "+PSPICE \n.include ../../ComponentModels/1n4148.spi\n.include ../../ComponentModels/2n3906.spi\n.include ../../ComponentModels/irf4905.spi\n\n*.DC V1 5 15 0.001\n.TRAN 0.5us 10ms\n // transient analysis for 10 ms in steps of 0.5 us (20,000 steps)\n.control\nrun\nplot VA VK VG Vbase\nplot VA-VK\nplot VA-Vbase VK-Vbase VK-VG\nplot -i(V1) i(V2)\n*plot VD*1000\nplot (VD2-VD)*1000 (VD3-VD)*1000 VD*100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"
- note removed: "+PSPICE \n.include ../ComponentModels/1n4148.spi\n.include ../ComponentModels/2n3906.spi\n.include ../ComponentModels/irf4905.spi\n\n*.DC V1 5 15 0.001\n.TRAN 0.05us 10ms\n // transient analysis for 10 ms in steps of 0.1 us (10,000 steps)\n.control\nrun\nplot VA VK VG Vbase\nplot VA-VK\nplot VA-Vbase VK-Vbase VK-VG\nplot -i(V1) i(V2)\n*plot VD*1000\nplot (VD2-VD)*1000 (VD3-VD)*1000 VD*1000\n"
Changed lines of the file:
@@
 encoding utf-8
 Sheet 1 1
-Title "XL4016X2"
-Date "2018-04-11"
-Rev "V3 minor corrections"
+Title "MOSFETdiodeDiscretes"
+Date "2018-05-24"
+Rev "V2"
 Comp "farmerkeith"
 Comment1 ""
@@
 $EndDescr
 Wire Wire Line
-	1800 1350 2850 1350
-Wire Wire Line
-	2850 1350 3150 1350
+	1800 1350 3150 1350
 $Comp
 L GND #PWR01
@@
 $EndComp
 Wire Wire Line
-	1800 3700 2850 3700
-Wire Wire Line
-	2850 3700 4700 3700
+	1800 3700 4700 3700
 Wire Wire Line
 	3400 1850 3150 1850
@@
 	2400 2600 2400 1150
 Text Notes 5250 2750 0    60   ~ 0
-+PSPICE \n.include ../ComponentModels/1n4148.spi\n.include ../ComponentModels/2n3906.spi\n.include ../ComponentModels/irf4905.spi\n\n*.DC V1 5 15 0.001\n.TRAN 0.05us 10ms\n // transient analysis for 10 ms in steps of 0.1 us (10,000 steps)\n.control\nrun\nplot VA VK  VG Vbase\nplot VA-VK\nplot VA-Vbase VK-Vbase VK-VG\nplot -i(V1) i(V2)\n*plot VD*1000\nplot (VD2-VD)*1000 (VD3-VD)*1000 VD*1000\n
++PSPICE \n.include ../../ComponentModels/1n4148.spi\n.include ../../ComponentModels/2n3906.spi\n.include ../../ComponentModels/irf4905.spi\n\n*.DC V1 5 15 0.001\n.TRAN 0.5us 10ms\n // transient analysis for 10 ms in steps of 0.5 us (20,000 steps)\n.control\nrun\nplot VA VK  VG Vbase\nplot VA-VK\nplot VA-Vbase VK-Vbase VK-VG\nplot -i(V1) i(V2)\n*plot VD*1000\nplot (VD2-VD)*1000 (VD3-VD)*1000 VD*1000\n
 $Comp
 L VSOURCE V1
@@
 $EndComp
 Wire Wire Line
-	3550 1350 3700 1350
-Wire Wire Line
-	3700 1350 4200 1350
+	3550 1350 4200 1350
 Connection ~ 3700 1350
 $Comp
@@
 VD3
 $Comp
-L IRF4905 Q1
+L IRF4905 XQ1
 U 1 1 5AF774ED
 P 3350 1450
-F 0 "Q1" V 3350 1600 50  0000 L CNN
+F 0 "XQ1" V 3350 1600 50  0000 L CNN
 F 1 "IRF4905" V 3600 1350 50  0000 L CNN
 F 2 "TO-220" H 3550 1375 50  0001 L CIN
 F 3 "" H 3350 1450 50  0001 L CNN
+F 4 "2,1,3" V 3350 1450 60  0001 C CNN "Spice_Node_Sequence"
 	1    3350 1450
 	0    -1   -1   0

Commit message: minor updates
Other:
- note removed: "pulse (9.50V 11.5V 2ms 0 0 5ms 10ms 0)\n\n.include ../ComponentModels/1n4148.spi\n.include ../ComponentModels/2n3906.spi\n.include ../ComponentModels/irf4905.spi\n\n*.TRAN 0.1us 10ms \n.DC V1 0 20 0.1\n // performs dc analysis; \n // sweeps V1 from 0 to 20 volts in steps of 0.1 volts\n.control\nrun\nplot VA VK VG Vbase\nplot VA-VK\nplot VA-Vbase VK-Vbase VK-VG\nplot -i(V1) i(V2)\n\n*plot diff=par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"
