File: PWMdriver/EnhancedDriverTIP/EnhancedDriverTIP.sch (KiCad schematic (older format))
At the start: 29 parts, among them Q1 IRFZ44N, Q2 2N3904, Q3 2N3904, Q4 TIP122, Q5 TIP125, Q6 2N3906

Commit message: updated for consistency with ng
Other:
- note added: "+PSPICE \n.model Zener30V D(bv=30v)\n* .include /home/guy/aProjects/circuits/ComponentModels/irfz44n.spi\n.include /home/guy/aProjects/circuits/ComponentModels/1n4148.spi\n.include /home/guy/aProjects/circuits/ComponentModels/32ctq030.spi\n*.include /home/guy/aProjects/circuits/ComponentModels/bc547.spi\n.include /home/guy/aProjects/circuits/ComponentModels/2n3904.spi\n.include /home/guy/aProject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"
- note removed: "+PSPICE \n.model Zener30V D(bv=30v)\n.include /home/guy/aProjects/circuits/ComponentModels/irfz44n.spi\n.include /home/guy/aProjects/circuits/ComponentModels/1n4148.spi\n.include /home/guy/aProjects/circuits/ComponentModels/32ctq030.spi\n*.include /home/guy/aProjects/circuits/ComponentModels/bc547.spi\n.include /home/guy/aProjects/circuits/ComponentModels/2n3904.spi\n.include /home/guy/aProjects/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"
Changed lines of the file:
@@
 Q1D
 Text Notes 7800 3850 0    60   ~ 0
-+PSPICE \n.model Zener30V D(bv=30v)\n.include /home/guy/aProjects/circuits/ComponentModels/irfz44n.spi\n.include /home/guy/aProjects/circuits/ComponentModels/1n4148.spi\n.include /home/guy/aProjects/circuits/ComponentModels/32ctq030.spi\n*.include /home/guy/aProjects/circuits/ComponentModels/bc547.spi\n.include /home/guy/aProjects/circuits/ComponentModels/2n3904.spi\n.include /home/guy/aProjects/circuits/ComponentModels/2n3906.spi\n*.include /home/guy/aProjects/circuits/ComponentModels/sd882.spi\n*.include /home/guy/aProjects/circuits/ComponentModels/sb772.spi\n.include /home/guy/aProjects/circuits/ComponentModels/tip122.spi\n.include /home/guy/aProjects/circuits/ComponentModels/tip125.spi\n.control\ntran 10ns 15us \nplot vin*8 q1g q1s vb\ntran 2ns 1.5us 0.9us \n*plot q1g vsl\nplot vpp1 q1d vbb\nplot (q1s-vsl)*1000  i(v1)\nplot vin*8 q1g q1s vb\nplot vin*8 q2b*10 q2c q2e vb\ntran 2ns 4.5us 4us \nplot vin*8 q1g q1s vb\nplot vin*8 q2b*10 q2c q2e vb\ntran 100ns 1ms \nplot I(V1)\nplot vpp1 vcl\ntran 10ns 1000us 980us\nplot I(V1)\nplot vin*8 q1g q1s vb\n.endc
++PSPICE \n.model Zener30V D(bv=30v)\n* .include /home/guy/aProjects/circuits/ComponentModels/irfz44n.spi\n.include /home/guy/aProjects/circuits/ComponentModels/1n4148.spi\n.include /home/guy/aProjects/circuits/ComponentModels/32ctq030.spi\n*.include /home/guy/aProjects/circuits/ComponentModels/bc547.spi\n.include /home/guy/aProjects/circuits/ComponentModels/2n3904.spi\n.include /home/guy/aProjects/circuits/ComponentModels/2n3906.spi\n*.include /home/guy/aProjects/circuits/ComponentModels/sd882.spi\n*.include /home/guy/aProjects/circuits/ComponentModels/sb772.spi\n*.include /home/guy/aProjects/circuits/ComponentModels/tip122.spi\n*.include /home/guy/aProjects/circuits/ComponentModels/tip125.spi\n.control\ntran 10ns 15us \nplot vin*8 q1g q1s vb\ntran 2ns 1.5us 0.9us \n*plot q1g vsl\nplot vpp1 q1d vbb\nplot (q1s-vsl)*1000  i(v1)\nplot vin*8 q1g q1s vb\nplot vin*8 q2b*10 q2c q2e vb\ntran 2ns 4.5us 4us \nplot vin*8 q1g q1s vb\nplot vin*8 q2b*10 q2c q2e vb\ntran 100ns 1ms \nplot I(V1)\nplot vpp1 vcl\ntran 10ns 1000us 980us\nplot I(V1)\nplot vin*8 q1g q1s vb\n.endc
 $Comp
 L R R10
